Commit message: Updated size of robot in URDF

File: description/robot_core.xacro (robot description, xacro)
@@ -1,5 +1,5 @@
 <?xml version="1.0"?>
 <robot xmlns:xacro="http://www.ros.org/wiki/xacro" >
-    <!-- <xacro:include filename="inertial_macros.xacro"/> -->
+    <xacro:include filename="inertial_macros.xacro"/>
     <material name="white">
         <color rgba="1 1 1 1" />
@@ -21,5 +21,5 @@
         <parent link="base_link"/>
         <child link="chassis"/>
-        <origin xyz="0 160 0"/>
+        <origin xyz="0 .160 0"/>
     </joint>
     <!-- Length: 310mm (approx),
@@ -30,16 +30,108 @@
     <link name="chassis">
         <visual>
-            <origin xyz="60 -228 0"/>
+            <origin xyz=".060 -.228 0"/>
             <geometry>
-                <mesh filename="file://$(find my_bot)/description/meshes/forklift_chassis.stl"/>
+                <mesh filename="file://$(find my_bot)/description/meshes/forklift_chassis.stl" scale=".001 .001 .001"/>
             </geometry>
             <material name="white"/>
         </visual>
         <collision>
-            <!-- <origin xyz="-10 1 0.25"/> -->
+            <origin xyz=".060 -.228 0"/>
             <geometry>
-                <mesh filename="file://$(find my_bot)/description/meshes/forklift_chassis.stl" />
+                <mesh filename="file://$(find my_bot)/description/meshes/forklift_chassis.stl" scale=".001 .001 .001 " />
             </geometry>
         </collision>
     </link>
+<!-- BACK LEFT WHEEL LINK -->
+    <joint name="back_left_wheel_joint" type="fixed">
+        <parent link="base_link"/>
+        <child link="back_left_wheel"/>
+        <origin xyz=".080 ${.168 - .040} -.005" rpy="-${pi/2} 0 -${pi/2}"/>
+        <axis xyz="0 0 -1"/>
+    </joint>
+    <link name="back_left_wheel">
+        <visual>
+            <geometry>
+                <cylinder radius="${.067/2}" length="0.0255"/>
+            </geometry>
+            <material name="blue"/>
+        </visual>
+        <collision>
+            <geometry>
+                <cylinder radius="${.067/2}" length="0.0255"/>
+            </geometry>
+        </collision>
+        <xacro:inertial_cylinder mass="10" length="0.0255" radius="${.067/2}">
+            <origin xyz="0 0 0" rpy="0 0 0"/>
+        </xacro:inertial_cylinder>
+    </link>
+<!-- BACK RIGHT WHEEL LINK -->
+    <joint name="back_right_wheel_joint" type="fixed">
+        <parent link="base_link"/>
+        <child link="back_right_wheel"/>
+        <origin xyz="-.080 ${.168 - .040} -.005" rpy="-${pi/2} 0 ${pi/2}"/>
+        <axis xyz="0 0 -1"/>
+    </joint>
+    <link name="back_right_wheel">
+        <visual>
+            <geometry>
+                <cylinder radius="${.067/2}" length="0.0255"/>
+            </geometry>
+            <material name="blue"/>
+        </visual>
+        <collision>
+            <geometry>
+                <cylinder radius="${.067/2}" length="0.0255"/>
+            </geometry>
+        </collision>
+        <xacro:inertial_cylinder mass="10" length="0.0255" radius="${.067/2}">
+            <origin xyz="0 0 0" rpy="0 0 0"/>
+        </xacro:inertial_cylinder>
+    </link>
+<!-- FRONT LEFT WHEEL LINK -->
+    <joint name="front_left_wheel_joint" type="fixed">
+        <parent link="base_link"/>
+        <child link="front_left_wheel"/>
+        <origin xyz=".080 -${.142 - (.067/2)} -.005" rpy="-${pi/2} 0 ${pi/2}"/>
+        <axis xyz="0 0 -1"/>
+    </joint>
+    <link name="front_left_wheel">
+        <visual>
+            <geometry>
+                <cylinder radius="${.067/2}" length="0.0255"/>
+            </geometry>
+            <material name="blue"/>
+        </visual>
+        <collision>
+            <geometry>
+                <cylinder radius="${.067/2}" length="0.0255"/>
+            </geometry>
+        </collision>
+        <xacro:inertial_cylinder mass="10" length="0.0255" radius="${.067/2}">
+            <origin xyz="0 0 0" rpy="0 0 0"/>
+        </xacro:inertial_cylinder>
+    </link>
+    <!-- FRONT RIGHT WHEEL LINK -->
+    <joint name="front_right_wheel_joint" type="fixed">
+        <parent link="base_link"/>
+        <child link="front_right_wheel"/>
+        <origin xyz="-.080 -${.142 - (.067/2)} -.005" rpy="-${pi/2} 0 ${pi/2}"/>
+        <axis xyz="0 0 -1"/>
+    </joint>
+    <link name="front_right_wheel">
+        <visual>
+            <geometry>
+                <cylinder radius="${.067/2}" length="0.0255"/>
+            </geometry>
+            <material name="blue"/>
+        </visual>
+        <collision>
+            <geometry>
+                <cylinder radius="${.067/2}" length="0.0255"/>
+            </geometry>
+        </collision>
+        <xacro:inertial_cylinder mass="10" length="0.0255" radius="${.067/2}">
+            <origin xyz="0 0 0" rpy="0 0 0"/>
+        </xacro:inertial_cylinder>
+    </link>
 </robot>

Commit message: Updated encoder counts

File: description/robot_core.xacro (robot description, xacro)
@@ -19,4 +19,11 @@
     <!-- BASE LINK -->
     <link name="base_link">
+    </link>
+    <joint name="base_footprint_joint" type="fixed">
+        <parent link="base_link"/>
+            <child link="base_footprint"/>
+            <origin xyz="0 0 0" rpy="0 0 0" />
+    </joint>
+    <link name="base_footprint">
     </link>
     <!-- CHASSIS LINK -->

File: description/ros2_control.xacro (robot description, xacro)
@@ -11,5 +11,5 @@
                 <param name="baud_rate">57600</param>
                 <param name="timeout">1000</param>
-                <param name="enc_counts_per_rev">12</param>
+                <param name="enc_counts_per_rev">24</param>
             </hardware>
             <joint name="left_wheel_joint">

Commit message: I rotated robot base by 90 degree

File: description/robot_core.xacro (robot description, xacro)
@@ -23,5 +23,5 @@
         <parent link="base_link"/>
             <child link="base_footprint"/>
-            <origin xyz="0 0 0" rpy="0 0 0" />
+            <origin xyz="0 0 0" rpy="0 0 -1.5708" />
     </joint>
     <link name="base_footprint">
