Commit message: Updated robot URDF

File: description/inertial_macros.xacro (robot description, xacro)
@@ -3,4 +3,13 @@
     <!-- Specify some standard inertial calculations https://en.wikipedia.org/wiki/List_of_moments_of_inertia -->
     <!-- These make use of xacro's mathematical functionality -->
+    <xacro:macro name="inertial_sphere" params="mass radius *origin">
+        <inertial>
+            <xacro:insert_block name="origin"/>
+            <mass value="${mass}" />
+            <inertia ixx="${(2/5) * mass * (radius*radius)}" ixy="0.0" ixz="0.0"
+                    iyy="${(2/5) * mass * (radius*radius)}" iyz="0.0"
+                    izz="${(2/5) * mass * (radius*radius)}" />
+        </inertial>
+    </xacro:macro>
     <xacro:macro name="inertial_cylinder" params="mass length radius *origin">
         <inertial>

File: description/lidar.xacro (robot description, xacro)
@@ -4,5 +4,6 @@
         <parent link="chassis"/>
         <child link="laser_frame"/>
-        <origin xyz="0 -0.14 0.18" rpy="0 0 ${pi}"/>
+        <!-- <origin xyz="0 -0.14 0.18" rpy="0 0 ${pi}"/> -->
+        <origin xyz="0 0.03 0.185" rpy="0 0 ${pi}"/>
     </joint>
     <link name="laser_frame">

File: description/robot_core.xacro (robot description, xacro)
@@ -23,5 +23,5 @@
         <parent link="base_link"/>
             <child link="base_footprint"/>
-            <origin xyz="0 0 0" rpy="0 0 -1.5708" />
+            <origin xyz="0 0 0" rpy="0 0 ${pi/2}" />
     </joint>
     <link name="base_footprint">
@@ -29,7 +29,6 @@
     <!-- CHASSIS LINK -->
     <joint name="chassis_joint" type="fixed">
-        <parent link="base_link"/>
+        <parent link="base_footprint"/>
         <child link="chassis"/>
-        <origin xyz="0 .160 0"/>
     </joint>
     <!-- Length= 310mm (approx),
@@ -40,5 +39,5 @@
     <link name="chassis">
         <visual>
-            <origin xyz=".060 -.228 0"/>
+            <origin xyz=".060 -0.060 0"/>
             <geometry>
                 <mesh filename="file://$(find my_bot)/description/meshes/forklift_chassis.stl" scale=".001 .001 .001"/>
@@ -47,5 +46,5 @@
         </visual>
         <collision>
-            <origin xyz=".060 -.228 0"/>
+            <origin xyz=".060 -0.060 0"/>
             <geometry>
                 <mesh filename="file://$(find my_bot)/description/meshes/forklift_chassis.stl" scale=".001 .001 .001 " />
@@ -59,6 +58,6 @@
     </link>
 <!-- BACK LEFT WHEEL LINK -->
-    <joint name="back_left_wheel_joint" type="fixed">
-        <parent link="base_link"/>
+    <joint name="back_left_wheel_joint" type="continuous">
+        <parent link="chassis"/>
         <child link="back_left_wheel"/>
         <origin xyz=".080 ${.168 - .040} -.005" rpy="-${pi/2} 0 -${pi/2}"/>
@@ -82,6 +81,6 @@
     </link>
 <!-- BACK RIGHT WHEEL LINK -->
-    <joint name="back_right_wheel_joint" type="fixed">
-        <parent link="base_link"/>
+    <joint name="back_right_wheel_joint" type="continuous">
+        <parent link="chassis"/>
         <child link="back_right_wheel"/>
         <origin xyz="-.080 ${.168 - .040} -.005" rpy="-${pi/2} 0 ${pi/2}"/>
@@ -104,49 +103,28 @@
         </xacro:inertial_cylinder>
     </link>
-<!-- FRONT LEFT WHEEL LINK -->
-    <joint name="front_left_wheel_joint" type="fixed">
-        <parent link="base_link"/>
-        <child link="front_left_wheel"/>
-        <origin xyz=".080 -${.142 - (.067/2)} -.005" rpy="-${pi/2} 0 ${pi/2}"/>
-        <axis xyz="0 0 -1"/>
+    <!-- CASTER WHEEL LINK -->
+ <joint name="caster_wheel_joint" type="fixed">
+        <parent link="chassis"/>
+        <child link="caster_wheel"/>
+        <origin xyz="0 -${.168 - .040} ${(-.067/2) + 0.0127}"/>
     </joint>
-    <link name="front_left_wheel">
+            <!-- For the z axis of the origin, I brought the castor wheel down by the radius of the back tires (hence -0.067/2) as they are on the same plane
+        but then I brought it up by it's own radius to make the bottom of the wheel to line up with the bottom of the back tires (hence + 0.0127)
+         -->
+    <link name="caster_wheel">
         <visual>
             <geometry>
-                <cylinder radius="${.067/2}" length="0.0255"/>
+                <sphere radius="0.0127"/>
             </geometry>
-            <material name="blue"/>
+            <material name="black"/>
         </visual>
         <collision>
             <geometry>
-                <cylinder radius="${.067/2}" length="0.0255"/>
+                <sphere radius="0"/>
             </geometry>
         </collision>
-        <xacro:inertial_cylinder mass="0.04" length="0.0255" radius="${.067/2}">
+        <xacro:inertial_sphere mass="0.1" radius="0.0127">
             <origin xyz="0 0 0" rpy="0 0 0"/>
-        </xacro:inertial_cylinder>
-    </link>
-    <!-- FRONT RIGHT WHEEL LINK -->
-    <joint name="front_right_wheel_joint" type="fixed">
-        <parent link="base_link"/>
-        <child link="front_right_wheel"/>
-        <origin xyz="-.080 -${.142 - (.067/2)} -.005" rpy="-${pi/2} 0 ${pi/2}"/>
-        <axis xyz="0 0 -1"/>
-    </joint>
-    <link name="front_right_wheel">
-        <visual>
-            <geometry>
-                <cylinder radius="${.067/2}" length="0.0255"/>
-            </geometry>
-            <material name="blue"/>
-        </visual>
-        <collision>
-            <geometry>
-                <cylinder radius="${.067/2}" length="0.0255"/>
-            </geometry>
-        </collision>
-        <xacro:inertial_cylinder mass="0.04" length="0.0255" radius="${.067/2}">
-            <origin xyz="0 0 0" rpy="0 0 0"/>
-        </xacro:inertial_cylinder>
+        </xacro:inertial_sphere>
     </link>
 </robot>
