Commit message: Updated lidar.xacro

File: description/lidar.xacro (robot description, xacro)
@@ -4,6 +4,5 @@
         <parent link="chassis"/>
         <child link="laser_frame"/>
-        <!-- <origin xyz="0 -0.14 0.18" rpy="0 0 ${pi}"/> -->
-        <origin xyz="0 0.03 0.185" rpy="0 0 ${pi}"/>
+        <origin xyz="0 0.03 0.185" rpy="0 0 -${pi/2}"/>
     </joint>
     <link name="laser_frame">

File: description/robot_core.xacro (robot description, xacro)
@@ -58,5 +58,5 @@
     </link>
 <!-- BACK LEFT WHEEL LINK -->
-    <joint name="back_left_wheel_joint" type="continuous">
+    <joint name="back_left_wheel_joint" type="fixed">
         <parent link="chassis"/>
         <child link="back_left_wheel"/>
@@ -81,5 +81,5 @@
     </link>
 <!-- BACK RIGHT WHEEL LINK -->
-    <joint name="back_right_wheel_joint" type="continuous">
+    <joint name="back_right_wheel_joint" type="fixed">
         <parent link="chassis"/>
         <child link="back_right_wheel"/>

File: description/ros2_control.xacro (robot description, xacro)
@@ -8,5 +8,5 @@
                 <param name="right_wheel_name">right_wheel_joint</param>
                 <param name="loop_rate">30</param>
-                <param name="device">/dev/ttyUSB0</param>
+                <param name="device">/dev/serial/by-id/usb-1a86_USB_Serial-if00-port0</param>
                 <param name="baud_rate">57600</param>
                 <param name="timeout">1000</param>
